File: rocket/rocket.kicad_pcb (KiCad board)
At the start: 4 copper layers, 30.5 x 38.1 mm, 41 parts, among them J1 Conn_02x04_Odd_Even, J2 BATT, J3 USB_C_Receptacle_USB2.0, J4 u.FL, SW1 SW_DPDT_x2, SW2 SW_SPST, U1 MCP73831-2ACL-OT, U2 XC6206P332MR, U3 NEO-6M_module, U4 RFM95W-915S2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

Commit message: Symbol, Footprint, and 3D libraries added
Parts:
- J1: footprint custom:PinSocket_2x04_P1.27mm_Horizontal_Straddle -> rocket_tracker:PinSocket_2x04_P1.27mm_Horizontal_Straddle
- J3: footprint custom:GCT_USB4110-GF-A -> rocket_tracker:GCT_USB4110-GF-A
- SW1: footprint custom:SW_DPDT_CK_JS202011JAQN -> rocket_tracker:SW_DPDT_CK_JS202011JAQN
- SW2: footprint custom:SW_Push_1P1T_KSS231 -> rocket_tracker:SW_Push_1P1T_KSS231
- U3: footprint custom:NEO-6M_module -> rocket_tracker:NEO-6M_module
- U7: footprint custom:LGA-24L_3x3.5mm_P0.43mm_Handsolder -> rocket_tracker:LGA-24L_3x3.5mm_P0.43mm_Handsolder
