File: rocket/rocket.sch (KiCad schematic (older format))
At the start: 41 parts, among them J1 Conn_02x04_Odd_Even, J2 BATT, J3 USB_C_Receptacle_USB2.0, J4 u.FL, SW1 SW_DPDT_x2, SW2 SW_SPST, U1 MCP73831-2ACL-OT, U2 XC6206P332MR, U3 NEO-6M_module, U4 RFM95W-915S2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

Commit message: Symbol, Footprint, and 3D libraries added
Parts:
- U3: footprint custom:NEO-6M_module -> rocket_tracker:NEO-6M_module; symbol custom:NEO-6M_module -> rocket_tracker:NEO-6M_module
Changed lines of the file:
@@
 $EndComp
 $Comp
-L custom:NEO-6M_module U3
+L rocket_tracker:NEO-6M_module U3
 U 1 1 5EF24A8A
 P 5500 2700
 F 0 "U3" H 5780 2721 50  0000 L CNN
 F 1 "NEO-6M_module" H 5780 2630 50  0000 L CNN
-F 2 "custom:NEO-6M_module" H 5950 3150 50  0001 C CNN
+F 2 "rocket_tracker:NEO-6M_module" H 5950 3150 50  0001 C CNN
 F 3 "" H 5500 2700 50  0001 C CNN
 F 4 "DIGIKEY" H 5500 2700 50  0001 C CNN "Supplier"
